File: files/wirings/wirings.kicad_sch (KiCad schematic)
At the start: 15 parts, among them P1 Motor12V, SW1 PWR Rocker, SW2 RST SW, U1 RPi4_Objective, U2 VL53L0/1XV2, U3 LSF02, U4 HW-688, U5 Heatsink+PWMFan

Commit message: 10072023
Parts:
- removed U2: VL53L0/1XV2, symbol Sensors and Others:VL53L0/1XV2
- added U?: E18-D80NK, symbol Sensors and Others:E18-D80NK
Connections:
- net at U3. (VREFB): now also R1. (VCC)
- net at R2. (VCC): now also R1. (VCC), U1. (VIN-); no longer U3. (VREFB)
- net at U1. (VIN-): now also SW1.1 (A); no longer U3. (VREFB)
- net at R1. (VCC): now also S1. (-); no longer U3. (VREFB)
- net at U1. (VIN-), U5. (VCC): now also U?. (VIN)
- net at U4. (VIN-): now also SW1.2 (B); no longer U1. (VIN-)
- new net: R2. (VCC), U3. (VREFB)
- new net: R1. (VCC), R2. (VCC), U1. (VIN-), U3. (VREFB)
- new net: D2.2 (A), U1. (VIN-), U3. (VREFB)
- new net: D3.2 (A), U1. (VIN-), U3. (VREFB)
- new net: D1.2 (A), U1. (VIN-), U3. (VREFB)
- new net: U1. (VIN-), U3. (VREFB) (x2)
- new net: U3. (VREFB), U?. (VIN)
- new net: U1. (VIN-), U5. (VCC)
- new net: U1. (VIN-), U5. (VCC), U?. (VIN)
- new net: P1. (-), R1. (VCC), R2. (VCC), S1. (-), U4. (VIN-), XBT1. (-)
- new net: R1. (VCC), R2. (VCC), U4. (VIN-), XBT1. (-)
- new net: U1. (VIN-), U4. (VIN-)
- no-connect marks 27 -> 24

Commit message: 10072023
Connections:
- net at U3. (VREFB): now also R1. (VCC)
- net at R2. (VCC): now also R1. (VCC), U1. (VIN-); no longer U3. (VREFB)
- net at U1. (VIN-): now also SW1.1 (A); no longer U3. (VREFB)
- net at U?. (VIN): now also U1. (VIN-), U5. (VCC); no longer U3. (VREFB)
- net at R1. (VCC): now also S1. (-); no longer U3. (VREFB)
- net at U4. (VIN-): now also SW1.2 (B); no longer U1. (VIN-)
- new net: R2. (VCC), U3. (VREFB)
- new net: R1. (VCC), R2. (VCC), U1. (VIN-), U3. (VREFB)
- new net: D2.2 (A), U1. (VIN-), U3. (VREFB)
- new net: D3.2 (A), U1. (VIN-), U3. (VREFB)
- new net: D1.2 (A), U1. (VIN-), U3. (VREFB)
- new net: U1. (VIN-), U3. (VREFB) (x2)
- new net: U3. (VREFB), U?. (VIN)
- new net: U1. (VIN-), U5. (VCC)
- new net: U1. (VIN-), U5. (VCC), U?. (VIN)
- new net: P1. (-), R1. (VCC), R2. (VCC), S1. (-), U4. (VIN-), XBT1. (-)
- new net: R1. (VCC), R2. (VCC), U4. (VIN-), XBT1. (-)
- new net: U1. (VIN-), U4. (VIN-)
