File: files/wirings/final.kicad_sch (KiCad schematic)
At the start: 15 parts, among them P1 Motor12V, SW1 PWR Rocker, SW2 RST SW, U1 RPi4_Objective, U2 VL53L0/1XV2, U3 LSF02, U4 HW-688, U5 Heatsink+PWMFan

Commit message: 23062023
Parts:
- removed U5: Heatsink+PWMFan, symbol Sensors and Others:Heatsink+PWMFan
- added U4: E18-D80NK, symbol Sensors and Others:E18-D80NK
- added U5: AJ-SR04M, symbol Sensors and Others:AJ-SR04M
- added U7: Heatsink+PWMFan, symbol Sensors and Others:Heatsink+PWMFan
- SW2: value RST SW -> SW_Push
- renumbered U4 to U6
Connections:
- net at U3. (VREFB): now also U1. (VIN-)
- net at R2. (VCC): now also R1. (VCC), U1. (VIN-); no longer U3. (VREFB)
- net at U1. (VIN-): now also SW1.1 (A); no longer U3. (VREFB)
- net at R1. (VCC): now also S1. (-); no longer U3. (VREFB)
- net at P1. (-), R2. (VCC): now also R1. (VCC), S1. (-), U6. (VIN-), XBT1. (-)
- net at U6. (VIN-): now also SW1.2 (B); no longer U1. (VIN-)
- new net: P1. (-), R2. (VCC)
- new net: D2.2 (A), U1. (VIN-), U2. (XSHUT), U3. (VREFB)
- new net: R2. (VCC), U3. (VREFB)
- new net: R1. (VCC), R2. (VCC), U1. (VIN-), U3. (VREFB)
- new net: D3.2 (A), U1. (VIN-), U3. (VREFB)
- new net: U3. (VREFB), U5. (VIN)
- new net: U3. (VREFB), U4. (VIN), U5. (VIN)
- new net: D1.2 (A), U1. (VIN-), U3. (VREFB)
- new net: R1. (VCC), U3. (VREFB)
- new net: U1. (VIN-), U3. (VREFB) (x2)
- new net: R1. (VCC), R2. (VCC), U6. (VIN-), XBT1. (-)
- new net: U1. (VIN-), U4. (VIN), U5. (VIN), U7. (VCC)
- new net: U1. (VIN-), U4. (VIN), U5. (VIN)
- new net: U1. (VIN-), U2. (XSHUT) (x4)
- new net: U1. (VIN-), U7. (VCC) (x2)
- new net: U1. (VIN-), U6. (VIN-)
- now unconnected: U2. (XSHUT), U2. (XSHUT), U2. (XSHUT), U2. (XSHUT), U2. (XSHUT)
- no-connect marks 27 -> 20

Commit message: 10072023
Connections:
- net at P1. (-), R2. (VCC): now also R1. (VCC), S1. (-), U6. (VIN-), XBT1. (-)
- net at U3. (VREFB): now also U1. (VIN-); no longer R2. (VCC)
- net at U5. (VIN): now also U1. (VIN-), U4. (VIN); no longer U3. (VREFB)
- net at R1. (VCC): now also S1. (-); no longer U3. (VREFB)
- net at U1. (VIN-): now also SW1.1 (A); no longer U3. (VREFB)
- net at U2. (XSHUT): no longer U1. (VIN-)
- net at U6. (VIN-): now also SW1.2 (B); no longer U1. (VIN-)
- new net: P1. (-), R2. (VCC)
- new net: D2.2 (A), U1. (VIN-), U2. (XSHUT), U3. (VREFB)
- new net: R2. (VCC), U3. (VREFB)
- new net: R1. (VCC), R2. (VCC), U1. (VIN-), U3. (VREFB)
- new net: D3.2 (A), U1. (VIN-), U3. (VREFB)
- new net: U3. (VREFB), U5. (VIN)
- new net: U3. (VREFB), U4. (VIN), U5. (VIN)
- new net: D1.2 (A), U1. (VIN-), U3. (VREFB)
- new net: R1. (VCC), U3. (VREFB)
- new net: U1. (VIN-), U3. (VREFB) (x2)
- new net: R1. (VCC), R2. (VCC), U6. (VIN-), XBT1. (-)
- new net: R1. (VCC), R2. (VCC), U1. (VIN-)
- new net: U1. (VIN-), U4. (VIN), U5. (VIN), U7. (VCC)
- new net: U1. (VIN-), U2. (XSHUT) (x4)
- new net: U1. (VIN-), U7. (VCC)
- new net: U1. (VIN-), U6. (VIN-)
- now unconnected: U2. (XSHUT), U2. (XSHUT), U2. (XSHUT), U2. (XSHUT)
