File: files/wirings/do1.wirings.kicad_sch (KiCad schematic)
At the start: 15 parts, among them P1 Motor12V, SW1 PWR Rocker, SW2 RST SW, U1 RPi4_Objective, U2 LSF02, U3 AJ-SR04M, U4 HW-688, U5 Heatsink+PWMFan

Commit message: 15072023
Connections:
- net at U2. (VREFB): now also R1. (VCC); no longer R2. (VCC)
- net at U3. (VIN): now also U1. (VIN-), U5. (VCC); no longer U2. (VREFB)
- net at U1. (VIN-): now also SW1.1 (A); no longer U2. (VREFB)
- net at R1. (VCC): now also S1. (-); no longer U2. (VREFB)
- net at U4. (VIN-): now also SW1.2 (B); no longer U1. (VIN-)
- new net: U1. (VIN-), U2. (VREFB) (x3)
- new net: R1. (VCC), R2. (VCC), U1. (VIN-), U2. (VREFB)
- new net: D2.2 (A), U1. (VIN-), U2. (VREFB)
- new net: D3.2 (A), U1. (VIN-), U2. (VREFB)
- new net: D1.2 (A), U1. (VIN-), U2. (VREFB)
- new net: R2. (VCC), U2. (VREFB)
- new net: U2. (VREFB), U3. (VIN) (x2)
- new net: U1. (VIN-), U5. (VCC)
- new net: U1. (VIN-), U3. (VIN), U5. (VCC)
- new net: R1. (VCC), R2. (VCC), U1. (VIN-)
- new net: U1. (VIN-), U4. (VIN-)
- new net: P1. (-), R1. (VCC), R2. (VCC), S1. (-), U4. (VIN-), XBT1. (-)
- new net: R1. (VCC), R2. (VCC), U4. (VIN-), XBT1. (-)
- no-connect marks 24 -> 27
Other:
- moved on the sheet: D1, D2, D3, P1, R1, R2, S1, SW1, SW2, U2, U3, U4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
