File: files/wirings/do2.wirings.kicad_sch (KiCad schematic)
At the start: 15 parts, among them P1 Motor12V, SW1 PWR Rocker, SW2 RST SW, U1 RPi4_Objective, U2 VL53L0/1XV2, U3 LSF02, U4 HW-688, U5 Heatsink+PWMFan

Commit message: 13072023
Parts:
- removed SW1: PWR Rocker, symbol Switch:SW_SPST
- removed U4: HW-688, symbol Battery Power and Management:HW-688
Connections:
- net at U3. (VREFB): now also R1. (VCC)
- net at R2. (VCC): now also R1. (VCC), U1. (VIN-); no longer U3. (VREFB)
- net at U1. (VIN-): no longer U3. (VREFB)
- net at R1. (VCC): now also S1. (-); no longer U3. (VREFB)
- net at U2. (XSHUT): now also U1. (VIN-)
- new net: R2. (VCC), U3. (VREFB)
- new net: R1. (VCC), R2. (VCC), U1. (VIN-), U3. (VREFB)
- new net: D2.2 (A), U1. (VIN-), U2. (XSHUT), U3. (VREFB)
- new net: D3.2 (A), U1. (VIN-), U3. (VREFB)
- new net: D1.2 (A), U1. (VIN-), U3. (VREFB)
- new net: U1. (VIN-), U3. (VREFB)
- new net: U1. (VIN-), U5. (VCC) (x2)
- new net: P1. (-), R1. (VCC), R2. (VCC), S1. (-), XBT1. (-)
- new net: R1. (VCC), R2. (VCC), XBT1. (-)
- new net: U1. (VIN-), U2. (XSHUT) (x3)
- now unconnected: U1. (VIN-), U1. (VIN-), U1. (VIN-), U1. (VIN-), U1. (VIN-), U1. (VIN-), U1. (VIN-), U1. (VIN-), U1. (VIN-), U1. (VIN-), U1. (VIN-), U1. (VIN-), U1. (VIN-)
- no-connect marks 27 -> 29
Changed lines of the file:
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@@
   (junction (at 175.26 45.466) (diameter 0) (color 0 0 0 0)
   )
-  (junction (at 189.357 66.294) (diameter 0) (color 0 0 0 0)
-  )
   (junction (at 175.26 60.833) (diameter 0) (color 0 0 0 0)
   )
@@
   )
   (junction (at 127 38.1) (diameter 0) (color 0 0 0 0)
-  )
-  (junction (at 175.26 65.532) (diameter 0) (color 0 0 0 0)
   )
   (junction (at 80.01 91.567) (diameter 0) (color 0 0 0 0)
@@
   (no_connect (at 75.057 76.327))
   (no_connect (at 75.057 71.247))
+  (no_connect (at 38.227 100.457))
   (no_connect (at 75.057 73.787))
   (no_connect (at 101.727 53.467))
@@
   (no_connect (at 75.057 61.087))
   (no_connect (at 38.227 61.087))
+  (no_connect (at 38.227 97.917))
   (wire (pts (xy 135.89 133.35) (xy 135.89 139.7))
     (stroke (width 0) (type default) (color 0 0 0 0))
@@
     (stroke (width 0) (type default) (color 0 0 0 0))
   )
-  (wire (pts (xy 36.83 119.38) (xy 145.923 119.38))
-    (stroke (width 0) (type default) (color 0 0 0 0))
-  )
   (wire (pts (xy 140.97 48.387) (xy 140.97 50.546))
     (stroke (width 0) (type default) (color 0 0 0 0))
@@
     (stroke (width 0) (type default) (color 0 0 0 0))
   )
-  (wire (pts (xy 163.703 119.38) (xy 175.26 119.38))
-    (stroke (width 0) (type default) (color 0 0 0 0))
-  )
   (wire (pts (xy 175.26 60.833) (xy 175.26 65.532))
     (stroke (width 0) (type default) (color 0 0 0 0))
@@
     (stroke (width 0) (type default) (color 0 0 0 0))
   )
-  (wire (pts (xy 35.56 97.917) (xy 38.227 97.917))
-    (stroke (width 0) (type default) (color 0 0 0 0))
-  )
   (wire (pts (xy 124.587 45.847) (xy 127 45.847))
     (stroke (width 0) (type default) (color 0 0 0 0))
@@
     (stroke (width 0) (type default) (color 0 0 0 0))
   )
-  (wire (pts (xy 175.26 119.38) (xy 175.26 65.532))
-    (stroke (width 0) (type default) (color 0 0 0 0))
-  )
   (wire (pts (xy 29.083 133.35) (xy 135.89 133.35))
     (stroke (width 0) (type default) (color 0 0 0 0))
@@
     (stroke (width 0) (type default) (color 0 0 0 0))
   )
-  (wire (pts (xy 121.793 127) (xy 121.793 116.84))
-    (stroke (width 0) (type default) (color 0 0 0 0))
-  )
   (wire (pts (xy 77.47 53.467) (xy 75.057 53.467))
     (stroke (width 0) (type default) (color 0 0 0 0))
@@
     (stroke (width 0) (type default) (color 0 0 0 0))
   )
-  (wire (pts (xy 163.703 116.84) (xy 189.357 116.84))
-    (stroke (width 0) (type default) (color 0 0 0 0))
-  )
-  (wire (pts (xy 135.89 116.84) (xy 145.923 116.84))
-    (stroke (width 0) (type default) (color 0 0 0 0))
-  )
   (wire (pts (xy 135.89 139.7) (xy 133.35 139.7))
     (stroke (width 0) (type default) (color 0 0 0 0))
@@
     (stroke (width 0) (type default) (color 0 0 0 0))
   )
-  (wire (pts (xy 35.56 116.84) (xy 35.56 97.917))
-    (stroke (width 0) (type default) (color 0 0 0 0))
-  )
   (wire (pts (xy 144.78 48.006) (xy 144.78 63.5))
     (stroke (width 0) (type default) (color 0 0 0 0))
@@
     (stroke (width 0) (type default) (color 0 0 0 0))
   )
-  (wire (pts (xy 36.83 100.457) (xy 36.83 119.38))
-    (stroke (width 0) (type default) (color 0 0 0 0))
-  )
   (wire (pts (xy 135.89 83.947) (xy 77.47 83.947))
     (stroke (width 0) (type default) (color 0 0 0 0))
@@
     (stroke (width 0) (type default) (color 0 0 0 0))
   )
-  (wire (pts (xy 133.35 127) (xy 135.89 127))
-    (stroke (width 0) (type default) (color 0 0 0 0))
-  )
   (wire (pts (xy 99.06 58.547) (xy 101.727 58.547))
     (stroke (width 0) (type default) (color 0 0 0 0))
@@
     (stroke (width 0) (type default) (color 0 0 0 0))
   )
-  (wire (pts (xy 189.357 116.84) (xy 189.357 66.294))
-    (stroke (width 0) (type default) (color 0 0 0 0))
-  )
   (wire (pts (xy 85.09 40.64) (xy 35.56 40.64))
     (stroke (width 0) (type default) (color 0 0 0 0))
@@
     (stroke (width 0) (type default) (color 0 0 0 0))
   )
-  (wire (pts (xy 135.89 127) (xy 135.89 116.84))
-    (stroke (width 0) (type default) (color 0 0 0 0))
-  )
   (wire (pts (xy 81.28 94.107) (xy 75.057 94.107))
     (stroke (width 0) (type default) (color 0 0 0 0))
@@
     (stroke (width 0) (type default) (color 0 0 0 0))
   )
-  (wire (pts (xy 121.793 116.84) (xy 35.56 116.84))
-    (stroke (width 0) (type default) (color 0 0 0 0))
-  )
   (wire (pts (xy 27.94 139.7) (xy 27.94 83.947))
     (stroke (width 0) (type default) (color 0 0 0 0))
@@
     (stroke (width 0) (type default) (color 0 0 0 0))
   )
-  (wire (pts (xy 38.227 100.457) (xy 36.83 100.457))
-    (stroke (width 0) (type default) (color 0 0 0 0))
-  )
   (wire (pts (xy 166.116 63.5) (xy 203.2 63.5))
     (stroke (width 0) (type default) (color 0 0 0 0))
   )
   (wire (pts (xy 33.02 120.65) (xy 115.57 120.65))
-    (stroke (width 0) (type default) (color 0 0 0 0))
-  )
-  (wire (pts (xy 123.19 127) (xy 121.793 127))
     (stroke (width 0) (type default) (color 0 0 0 0))
   )
@@
     (pin "")
   )
-  (symbol (lib_id "Battery Power and Management:HW-688") (at 154.813 118.11 0) (mirror y) (unit 1)
-    (in_bom yes) (on_board yes)
-    (property "Reference" "U4" (id 0) (at 154.813 113.157 0))
-    (property "Value" "HW-688" (id 1) (at 154.813 123.19 0))
-    (property "Footprint" "" (id 2) (at 154.813 118.11 0)
-      (effects (font (size 1.27 1.27)) hide)
-    )
-    (property "Datasheet" "" (id 3) (at 154.813 118.11 0)
-      (effects (font (size 1.27 1.27)) hide)
-    )
-    (pin "")
-    (pin "")
-    (pin "")
-    (pin "")
-  )
-  (symbol (lib_id "Switch:SW_SPST") (at 128.27 127 0) (unit 1)
-    (in_bom yes) (on_board yes)
-    (property "Reference" "SW1" (id 0) (at 128.27 123.825 0))
-    (property "Value" "PWR Rocker" (id 1) (at 128.27 130.302 0))
-    (property "Footprint" "" (id 2) (at 128.27 127 0)
-      (effects (font (size 1.27 1.27)) hide)
-    )
-    (property "Datasheet" "~" (id 3) (at 128.27 127 0)
-      (effects (font (size 1.27 1.27)) hide)
-    )
-    (pin "1")
-    (pin "2")
-  )
   (sheet_instances
     (path "/" (page "1"))
@@
       (reference "S1") (unit 1) (value "SolenoidValve12V") (footprint "")
     )
-    (path "/f2092351-0de8-4220-9643-a536771f37ae"
-      (reference "SW1") (unit 1) (value "PWR Rocker") (footprint "")
-    )
     (path "/493b5bcf-cb2c-4242-b60e-ed4afd6da774"
       (reference "SW2") (unit 1) (value "RST SW") (footprint "")
@@
       (reference "U3") (unit 1) (value "LSF02") (footprint "")
     )
-    (path "/f047e73d-f428-49a5-a42a-a4f26e019f75"
-      (reference "U4") (unit 1) (value "HW-688") (footprint "")
-    )
     (path "/28cfc313-5404-4ce3-b4ce-5c6fbe3a699d"

Commit message: 15072023
Parts:
- removed U1: RPi4_Objective, symbol Raspberry Pi 4:RPi4_Objective
- added U1: ZeroLiPo, symbol Battery Power and Management:ZeroLiPo
- added U2: RPi4_Objective, symbol Raspberry Pi 4:RPi4_Objective
- added XBP1: ICR18650-JST2P-PACK, symbol Battery Power and Management:ICR18650-JST2P-PACK
- renumbered SW2 to SW1, U2 to U3, U3 to U4
Connections:
- net at U4. (VREFB): now also R1. (VCC)
- net at R2. (VCC): now also P1. (-); no longer U4. (VREFB)
- net at D3.2 (A), U4. (VREFB): now also U2. (VIN-)
- net at D1.2 (A), U4. (VREFB): now also U2. (VIN-)
- net at R1. (VCC): now also S1. (-); no longer U4. (VREFB)
- net at U5. (VCC): now also U1. (P7(LB)), U2. (VIN-)
- net at D1.1 (K), D2.1 (K), D3.1 (K): now also U2. (VIN-)
- net at SW1.1: now also U2. (VIN-)
- net at SW1.2: now also U2. (VIN-)
- new net: U2. (VIN-), U4. (VREFB)
- new net: R1. (VCC), R2. (VCC), U1. (P7(LB)), U2. (VIN-), U4. (VREFB)
- new net: D2.2 (A), U2. (VIN-), U3. (XSHUT), U4. (VREFB)
- new net: R2. (VCC), U4. (VREFB)
- new net: U2. (VIN-), U5. (VCC) (x2)
- new net: R1. (VCC), R2. (VCC), U2. (VIN-)
- new net: U2. (VIN-), U3. (XSHUT) (x4)
- new net: P1. (-), R1. (VCC), R2. (VCC), S1. (-), XBT1. (-)
- new net: R1. (VCC), R2. (VCC), XBT1. (-)
- new net: U1. (P7(LB)), XBP1. (-) (x2)
- now unconnected: U3. (XSHUT), U3. (XSHUT), U3. (XSHUT), U3. (XSHUT), U3. (XSHUT)
- no-connect marks 29 -> 33
Other:
- moved on the sheet: D1, D2, D3, P1, R1, R2, S1, SW1, U3, U4, U5, XBT1
