File: files/wirings/final.wirings.kicad_sch (KiCad schematic)
At the start: 13 parts, among them P1 Motor12V, SW1 RST SW, U1 RPi4_Objective, U2 VL53L0/1XV2, U3 LSF02, U4 Heatsink+PWMFan

Commit message: 13072023
Parts:
- removed SW1: RST SW, symbol Switch:SW_Push
- removed U4: Heatsink+PWMFan, symbol Sensors and Others:Heatsink+PWMFan
- added SW1: PWR Rocker, symbol Switch:SW_SPST
- added SW2: SW_Push, symbol Switch:SW_Push
- added U6: HW-688, symbol Battery Power and Management:HW-688
- added U7: Heatsink+PWMFan, symbol Sensors and Others:Heatsink+PWMFan
Connections:
- net at U3. (VREFB): now also U1. (VIN-)
- net at R2. (VCC): now also R1. (VCC), U1. (VIN-); no longer U3. (VREFB)
- net at U1. (VIN-): now also SW1.1 (A); no longer U3. (VREFB)
- net at R1. (VCC): now also S1. (-); no longer U3. (VREFB)
- net at P1. (-), R2. (VCC): now also R1. (VCC), S1. (-), XBT1. (-), U6. (VIN-)
- new net: P1. (-), R2. (VCC)
- new net: D2.2 (A), U1. (VIN-), U2. (XSHUT), U3. (VREFB)
- new net: R2. (VCC), U3. (VREFB)
- new net: R1. (VCC), R2. (VCC), U1. (VIN-), U3. (VREFB)
- new net: D3.2 (A), U1. (VIN-), U3. (VREFB)
- new net: D1.2 (A), U1. (VIN-), U3. (VREFB)
- new net: R1. (VCC), U3. (VREFB)
- new net: R1. (VCC), R2. (VCC), U6. (VIN-), XBT1. (-)
- new net: SW2.1, U1. (VIN-)
- new net: SW2.2, U1. (VIN-)
- new net: U1. (VIN-), U2. (XSHUT) (x4)
- new net: U1. (VIN-), U7. (VCC) (x3)
- new net: U1. (VIN-), U6. (VIN-)
- new net: SW1.2 (B), U6. (VIN-)
- now unconnected: U2. (XSHUT), U2. (XSHUT), U2. (XSHUT), U2. (XSHUT), U2. (XSHUT)
- no-connect marks 29 -> 27

Commit message: 15072023
Parts:
- renumbered U6 to U4, U7 to U5
Connections:
- net at P1. (-), R2. (VCC): now also R1. (VCC), S1. (-), U4. (VIN-), XBT1. (-)
- net at U3. (VREFB): now also R1. (VCC)
- net at R2. (VCC): now also R1. (VCC), U4. (VIN-), XBT1. (-); no longer U3. (VREFB)
- net at R1. (VCC): now also S1. (-); no longer U3. (VREFB)
- net at U1. (VIN-): now also SW1.1 (A); no longer U3. (VREFB)
- net at U2. (XSHUT): no longer U1. (VIN-)
- net at U4. (VIN-): now also SW1.2 (B); no longer U1. (VIN-)
- new net: P1. (-), R2. (VCC)
- new net: D2.2 (A), U1. (VIN-), U2. (XSHUT), U3. (VREFB)
- new net: R2. (VCC), U3. (VREFB)
- new net: R1. (VCC), R2. (VCC), U1. (VIN-), U3. (VREFB)
- new net: D3.2 (A), U1. (VIN-), U3. (VREFB)
- new net: U1. (VIN-), U3. (VREFB)
- new net: D1.2 (A), U1. (VIN-), U3. (VREFB)
- new net: R1. (VCC), R2. (VCC), U1. (VIN-)
- new net: U1. (VIN-), U2. (XSHUT) (x4)
- new net: U1. (VIN-), U5. (VCC) (x2)
- new net: U1. (VIN-), U4. (VIN-)
- now unconnected: U2. (XSHUT), U2. (XSHUT), U2. (XSHUT), U2. (XSHUT)
- no-connect marks 27 -> 30
